File: MacroPad.kicad_sch (KiCad schematic)
At the start: 36 parts, among them J1 Conn_01x04_Socket, SW1 SW_Push_45deg, SW10 SW_Push_45deg, SW11 SW_Push_45deg, SW12 SW_Push_45deg, SW13 SW_Push_45deg, SW14 SW_Push_45deg, SW15 SW_Push_45deg, SW16 SW_Push_45deg, SW17 RotaryEncoder_Switch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

Commit message: Added models & footprints to the repo
Parts:
- A1: footprint Module:RaspberryPi_Pico_Common_THT -> SillyPad:RaspberryPi_Pico_Common_THT
- J1: footprint promicro:MODULE_DM-OLED096-636 -> SillyPad:MODULE_DM-OLED096-636
- SW1, SW10, SW11, SW12, SW13, SW14, SW15, SW16, SW2, SW3, SW4, SW5, SW6, SW7, SW8, SW9: footprint PCM_Switch_Keyboard_Cherry_MX:SW_Cherry_MX_Plate_1.00u -> SillyPad:SW_Cherry_MX_Plate_1.00u
Changed lines of the file:
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@@
 			)
 		)
-		(property "Footprint" "promicro:MODULE_DM-OLED096-636"
+		(property "Footprint" "SillyPad:MODULE_DM-OLED096-636"
 			(at 52.07 36.83 0)
 			(effects
@@
 			)
 		)
-		(property "Footprint" "PCM_Switch_Keyboard_Cherry_MX:SW_Cherry_MX_Plate_1.00u"
+		(property "Footprint" "SillyPad:SW_Cherry_MX_Plate_1.00u"
 			(at 121.92 113.03 0)
 			(effects
@@
 			)
 		)
-		(property "Footprint" "PCM_Switch_Keyboard_Cherry_MX:SW_Cherry_MX_Plate_1.00u"
+		(property "Footprint" "SillyPad:SW_Cherry_MX_Plate_1.00u"
 			(at 121.92 91.44 0)
 			(effects
@@
 			)
 		)
-		(property "Footprint" "PCM_Switch_Keyboard_Cherry_MX:SW_Cherry_MX_Plate_1.00u"
+		(property "Footprint" "SillyPad:SW_Cherry_MX_Plate_1.00u"
 			(at 105.41 91.44 0)
 			(effects
@@
 			)
 		)
-		(property "Footprint" "PCM_Switch_Keyboard_Cherry_MX:SW_Cherry_MX_Plate_1.00u"
+		(property "Footprint" "SillyPad:SW_Cherry_MX_Plate_1.00u"
 			(at 138.43 113.03 0)
 			(effects
@@
 			)
 		)
-		(property "Footprint" "PCM_Switch_Keyboard_Cherry_MX:SW_Cherry_MX_Plate_1.00u"
+		(property "Footprint" "SillyPad:SW_Cherry_MX_Plate_1.00u"
 			(at 154.94 134.62 0)
 			(effects
@@
 			)
 		)
-		(property "Footprint" "Module:RaspberryPi_Pico_Common_THT"
+		(property "Footprint" "SillyPad:RaspberryPi_Pico_Common_THT"
 			(at 53.34 144.78 0)
 			(effects
@@
 			)
 		)
-		(property "Footprint" "PCM_Switch_Keyboard_Cherry_MX:SW_Cherry_MX_Plate_1.00u"
+		(property "Footprint" "SillyPad:SW_Cherry_MX_Plate_1.00u"
 			(at 154.94 69.85 0)
 			(effects
@@
 			)
 		)
-		(property "Footprint" "PCM_Switch_Keyboard_Cherry_MX:SW_Cherry_MX_Plate_1.00u"
+		(property "Footprint" "SillyPad:SW_Cherry_MX_Plate_1.00u"
 			(at 121.92 134.62 0)
 			(effects
@@
 			)
 		)
-		(property "Footprint" "PCM_Switch_Keyboard_Cherry_MX:SW_Cherry_MX_Plate_1.00u"
+		(property "Footprint" "SillyPad:SW_Cherry_MX_Plate_1.00u"
 			(at 105.41 134.62 0)
 			(effects
@@
 			)
 		)
-		(property "Footprint" "PCM_Switch_Keyboard_Cherry_MX:SW_Cherry_MX_Plate_1.00u"
+		(property "Footprint" "SillyPad:SW_Cherry_MX_Plate_1.00u"
 			(at 121.92 69.85 0)
 			(effects
@@
 			)
 		)
-		(property "Footprint" "PCM_Switch_Keyboard_Cherry_MX:SW_Cherry_MX_Plate_1.00u"
+		(property "Footprint" "SillyPad:SW_Cherry_MX_Plate_1.00u"
 			(at 105.41 69.85 0)
 			(effects
@@
 			)
 		)
-		(property "Footprint" "PCM_Switch_Keyboard_Cherry_MX:SW_Cherry_MX_Plate_1.00u"
+		(property "Footprint" "SillyPad:SW_Cherry_MX_Plate_1.00u"
 			(at 105.41 113.03 0)
 			(effects
@@
 			)
 		)
-		(property "Footprint" "PCM_Switch_Keyboard_Cherry_MX:SW_Cherry_MX_Plate_1.00u"
+		(property "Footprint" "SillyPad:SW_Cherry_MX_Plate_1.00u"
 			(at 154.94 113.03 0)
 			(effects
@@
 			)
 		)
-		(property "Footprint" "PCM_Switch_Keyboard_Cherry_MX:SW_Cherry_MX_Plate_1.00u"
+		(property "Footprint" "SillyPad:SW_Cherry_MX_Plate_1.00u"
 			(at 154.94 91.44 0)
 			(effects
@@
 			)
 		)
-		(property "Footprint" "PCM_Switch_Keyboard_Cherry_MX:SW_Cherry_MX_Plate_1.00u"
+		(property "Footprint" "SillyPad:SW_Cherry_MX_Plate_1.00u"
 			(at 138.43 91.44 0)
 			(effects
@@
 			)
 		)
-		(property "Footprint" "PCM_Switch_Keyboard_Cherry_MX:SW_Cherry_MX_Plate_1.00u"
+		(property "Footprint" "SillyPad:SW_Cherry_MX_Plate_1.00u"
 			(at 138.43 134.62 0)
 			(effects
@@
 			)
 		)
-		(property "Footprint" "PCM_Switch_Keyboard_Cherry_MX:SW_Cherry_MX_Plate_1.00u"
+		(property "Footprint" "SillyPad:SW_Cherry_MX_Plate_1.00u"
 			(at 138.43 69.85 0)
 			(effects
